File: hardware/STR-21-007-SLAChamberHeater.kicad_pcb (KiCad board)
At the start: 4 copper layers, 60 x 25 mm, 56 parts, among them J101 2.5mm, J301 HEATER, J302 FAN, Q101 RU30L30M3, Q301 BSS138, Q302 RU30L30M3, Q303 RU3070M3, Q304 BSS138, SW201 SW_Push, SW202 SW_Push, SW401 SW_Push, U101 MP2359DJ-LF-Z, U201 ESP32-C3-MINI-1-N4, U202 USBLC6-2SC6, U301 LM75BDP

Commit message: DRC
Other:
- board text added: "FUSE"
Changed lines of the file:
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@@
     (property "Sheetfile" "Power.kicad_sch")
     (property "Sheetname" "[1] Power")
-    (attr through_hole)
+    (attr smd)
     (fp_text reference "U101" (at 0 -5.15 90) (layer "F.Fab") hide
       (effects (font (size 1 1) (thickness 0.15)))
@@
       (effects (font (size 1 1) (thickness 0.15)))
     )
-    (fp_circle (center 2.42 -1.33) (end 2.73 -1.33) (layer "F.Paste") (width 0.63) (fill none))
-    (fp_circle (center -2.42 -1.33) (end -2.11 -1.33) (layer "F.Paste") (width 0.63) (fill none))
+    (fp_line (start -3.78 2.78) (end -3.78 3.4) (layer "F.SilkS") (width 0.25))
+    (fp_line (start 3.8 0.16) (end 3.8 0.14) (layer "F.SilkS") (width 0.25))
+    (fp_line (start 3.36 -1.56) (end 3.8 -1.56) (layer "F.SilkS") (width 0.25))
+    (fp_line (start 3.8 3.375) (end 3.8 2.78) (layer "F.SilkS") (width 0.25))
     (fp_line (start -3.78 -1.56) (end -3.23 -1.56) (layer "F.SilkS") (width 0.25))
-    (fp_line (start -3.78 3.69) (end -4.12 4.03) (layer "F.SilkS") (width 0.25))
     (fp_line (start 3.8 -1.56) (end 3.8 0.14) (layer "F.SilkS") (width 0.25))
-    (fp_line (start 4.18 4.03) (end 3.8 3.65) (layer "F.SilkS") (width 0.25))
-    (fp_line (start 3.36 -1.56) (end 3.8 -1.56) (layer "F.SilkS") (width 0.25))
-    (fp_line (start -3.78 3.69) (end 3.8 3.69) (layer "F.SilkS") (width 0.25))
-    (fp_line (start -4.12 4.03) (end 4.01 4.03) (layer "F.SilkS") (width 0.25))
-    (fp_line (start 3.8 3.65) (end 3.8 2.78) (layer "F.SilkS") (width 0.25))
-    (fp_line (start -3.78 2.78) (end -3.78 3.69) (layer "F.SilkS") (width 0.25))
-    (fp_line (start 4.01 4.03) (end 4.18 4.03) (layer "F.SilkS") (width 0.25))
-    (fp_line (start 3.8 0.16) (end 3.8 0.14) (layer "F.SilkS") (width 0.25))
     (fp_line (start -3.78 -1.56) (end -3.78 0.15) (layer "F.SilkS") (width 0.25))
     (fp_circle (center -4 -1.58) (end -3.97 -1.58) (layer "F.Fab") (width 0.06) (fill none))
@@
     (pad "0" thru_hole oval (at -3.6 1.47 180) (size 1.3 2.2) (drill oval 0.700024 1.500124) (layers *.Cu *.Mask)
       (pinfunction "SHLD") (pintype "input+no_connect"))
+    (pad "0" thru_hole oval (at 3.6 1.47 180) (size 1.3 2.2) (drill oval 0.700024 1.500124) (layers *.Cu *.Mask)
+      (pinfunction "SHLD") (pintype "input+no_connect"))
     (pad "0" thru_hole circle (at 2.42 -1.33 180) (size 1.25 1.25) (drill 0.700024) (layers *.Cu *.Mask)
-      (pinfunction "SHLD") (pintype "input+no_connect"))
-    (pad "0" thru_hole oval (at 3.6 1.47 180) (size 1.3 2.2) (drill oval 0.700024 1.500124) (layers *.Cu *.Mask)
       (pinfunction "SHLD") (pintype "input+no_connect"))
     (pad "1" smd rect (at -1.31 -1.47 180) (size 0.45 1.25) (layers "F.Cu" "F.Paste" "F.Mask")
@@
     )
     (fp_line (start 2.525 1.181) (end 2.431 1.274) (layer "F.SilkS") (width 0.12))
-    (fp_line (start -1.81 -3.16) (end -1.81 4.56) (layer "F.SilkS") (width 0.12))
+    (fp_line (start -1.81 -3.16) (end -1.81 4.1) (layer "F.SilkS") (width 0.12))
     (fp_line (start 4.775 -1.069) (end 4.646 -0.941) (layer "F.SilkS") (width 0.12))
     (fp_line (start -1.81 3) (end 5.31 3) (layer "F.SilkS") (width 0.12))
-    (fp_line (start -2.05 4.8) (end -1.65 4.8) (layer "F.SilkS") (width 0.12))
-    (fp_line (start -2.05 4.16) (end -2.05 4.8) (layer "F.SilkS") (width 0.12))
     (fp_line (start 4.57 -1.275) (end 4.476 -1.181) (layer "F.SilkS") (width 0.12))
     (fp_line (start -1.81 4.1) (end 5.31 4.1) (layer "F.SilkS") (width 0.12))
     (fp_line (start -1.81 -3.16) (end 5.31 -3.16) (layer "F.SilkS") (width 0.12))
-    (fp_line (start -1.81 4.56) (end 5.31 4.56) (layer "F.SilkS") (width 0.12))
     (fp_line (start 2.355 0.941) (end 2.226 1.069) (layer "F.SilkS") (width 0.12))
-    (fp_line (start 5.31 -3.16) (end 5.31 4.56) (layer "F.SilkS") (width 0.12))
+    (fp_line (start 5.31 -3.16) (end 5.31 4.1) (layer "F.SilkS") (width 0.12))
     (fp_arc (start 0.890264 1.424721) (mid 0.463071 1.61492) (end 0 1.68) (layer "F.SilkS") (width 0.12))
     (fp_arc (start 1.425504 -0.890193) (mid 1.680626 0.000476) (end 1.425 0.891) (layer "F.SilkS") (width 0.12))
@@
       (effects (font (size 1 1) (thickness 0.15)))
     )
-    (fp_line (start 5.31 -3.16) (end 5.31 4.56) (layer "F.SilkS") (width 0.12))
-    (fp_line (start -2.05 4.16) (end -2.05 4.8) (layer "F.SilkS") (width 0.12))
-    (fp_line (start -1.81 4.56) (end 5.31 4.56) (layer "F.SilkS") (width 0.12))
+    (fp_line (start 5.31 -3.16) (end 5.31 4.1) (layer "F.SilkS") (width 0.12))
     (fp_line (start -1.81 4.1) (end 5.31 4.1) (layer "F.SilkS") (width 0.12))
     (fp_line (start 4.57 -1.275) (end 4.476 -1.181) (layer "F.SilkS") (width 0.12))
     (fp_line (start -1.81 3) (end 5.31 3) (layer "F.SilkS") (width 0.12))
     (fp_line (start 2.525 1.181) (end 2.431 1.274) (layer "F.SilkS") (width 0.12))
-    (fp_line (start -1.81 -3.16) (end -1.81 4.56) (layer "F.SilkS") (width 0.12))
-    (fp_line (start -2.05 4.8) (end -1.65 4.8) (layer "F.SilkS") (width 0.12))
+    (fp_line (start -1.81 -3.16) (end -1.81 4.1) (layer "F.SilkS") (width 0.12))
     (fp_line (start 4.775 -1.069) (end 4.646 -0.941) (layer "F.SilkS") (width 0.12))
     (fp_line (start 2.355 0.941) (end 2.226 1.069) (layer "F.SilkS") (width 0.12))
@@
     (effects (font (size 1 1) (thickness 0.15)))
   )
+  (gr_text "FUSE" (at 154.175 86.35 90) (layer "F.SilkS")
+    (effects (font (size 1 1) (thickness 0.15)))
+  )
